File: first-keep-pcb.kicad_pcb (KiCad board)
At the start: 2 copper layers, 77 x 38.1 mm, 24 parts, among them SW1 SW_Push, U1 ATmega32U4-AU, Y1 16MHz

Commit message: Added routing
Parts:
- moved C7 4.82 mm to (95.2, 88.1), turned to 270 degrees
- moved SW1 0.51 mm to (85.7, 92.6)
- turned F1 to 90 degrees
- turned R3 to 270 degrees
Routing:
- net GND: track 0.00 -> 148.1 mm
- net +5V: track 0.00 -> 104.5 mm, vias 0 -> 5
- net COL1: track 0.00 -> 52.3 mm
- net ROW1: track 0.00 -> 50.7 mm
- net ROW0: track 0.00 -> 46.9 mm
- net COL0: track 0.00 -> 32.9 mm
- net Net-(R3-Pad2): track 0.00 -> 32.2 mm, vias 0 -> 2
- net Net-(R1-Pad1): track 0.00 -> 22.7 mm
- net Net-(R2-Pad1): track 0.00 -> 21.5 mm
- net Net-(C4-Pad1): track 0.00 -> 13.3 mm
- net VCC: track 0.00 -> 11.2 mm
- net Net-(C3-Pad1): track 0.00 -> 10.3 mm
- net Net-(D4-Pad2): track 0.00 -> 6.62 mm
- net Net-(D3-Pad2): track 0.00 -> 6.62 mm
- net Net-(D2-Pad2): track 0.00 -> 6.62 mm
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Other:
- net class Default: trace_width 0.25 -> 0.254
- net class Power added: clearance 0.2, trace_width 0.381, via_dia 0.8, via_drill 0.4

Commit message: Added custom flair
Routing:
- added copper zone on B.Cu, net GND
Other:
- board text added: "Sup bitches"
Changed lines of the file:
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@@
   (general
     (thickness 1.6)
-    (drawings 10)
+    (drawings 11)
     (tracks 180)
     (zones 0)
@@
       (rotate (xyz 0 0 0))
     )
+  )
+  (gr_text "Sup bitches" (at 111.379 95.631) (layer F.SilkS)
+    (effects (font (size 1 1) (thickness 0.15) italic))
   )
   (gr_line (start 77.7875 96.04375) (end 77.7875 93.6625) (layer Edge.Cuts) (width 0.05))
@@
   (segment (start 110.49125 84.1525) (end 110.475 84.16875) (width 0.254) (layer B.Cu) (net 20))
   (segment (start 114.3 84.1525) (end 110.49125 84.1525) (width 0.254) (layer B.Cu) (net 20))
+  (zone (net 1) (net_name GND) (layer B.Cu) (hatch edge 0.508)
+    (connect_pads (clearance 0.508))
+    (min_thickness 0.254)
+    (fill yes (arc_segments 32) (thermal_gap 0.508) (thermal_bridge_width 0.508))
+    (polygon
+      (pts
+        (xy 116.713 97.663) (xy 77.597 97.663) (xy 77.724 59.563) (xy 116.713 59.563)
+      )
+    )
+  )
 )
